Commit message: feat: add jsw/st oint trajectory for ML leg

File: Models/Hexapod_mockup.urdf (robot description, URDF)
Before this commit: robot Hexapod_mockup.SLDASM, 27 links, 26 joints
Links:
- link BaseLink: geometry collision mesh filename=file:///home/tanawatp/Documents/Hexapod/PhysicalAI_modellin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; visual mesh filename=file:///home/tanawatp/Documents/Hexapod/PhysicalAI_modellin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
- link front_left_Endeffector: mass 8.67837417907314 -> None; geometry collision sphere radius=0.005; visual sphere radius=0.005
- link front_right_Endeffector: mass 8.67837417907314 -> None; geometry collision sphere radius=0.005; visual sphere radius=0.005
- link middle_left_Endeffector: mass 8.67837417907314 -> None; geometry collision sphere radius=0.005; visual sphere radius=0.005
- link middle_right_Endeffector: mass 8.67837417907314 -> None; geometry collision sphere radius=0.005; visual sphere radius=0.005
- link rear_left_Endeffector: mass 8.67837417907314 -> None; geometry collision sphere radius=0.005; visual sphere radius=0.005
- link rear_right_Endeffector: mass 8.67837417907314 -> None; geometry collision sphere radius=0.005; visual sphere radius=0.005
Joints:
- joint base_x_axis_offset: limit lower=-3.14 upper=3.14 effort=0 velocity=0 -> lower=-3.14 upper=3.14 effort=5 velocity=0
- joint base_z_axis_offset: limit lower=-3.14 upper=3.14 effort=0 velocity=0 -> lower=-3.14 upper=3.14 effort=5 velocity=0
- joint front_left_HeelJoint: limit lower=-3.14 upper=3.14 effort=0 velocity=0 -> lower=-3.14 upper=3.14 effort=5 velocity=0
- joint front_left_HipJoint: limit lower=-3.14 upper=3.14 effort=0 velocity=0 -> lower=-3.14 upper=3.14 effort=5 velocity=0
- joint front_left_KneeJoint: limit lower=-3.14 upper=3.14 effort=0 velocity=0 -> lower=-3.14 upper=3.14 effort=5 velocity=0
- joint front_right_HeelJoint: limit lower=-3.14 upper=3.14 effort=0 velocity=0 -> lower=-3.14 upper=3.14 effort=5 velocity=0
- joint front_right_HipJoint: limit lower=-3.14 upper=3.14 effort=0 velocity=0 -> lower=-3.14 upper=3.14 effort=5 velocity=0
- joint front_right_KneeJoint: limit lower=-3.14 upper=3.14 effort=0 velocity=0 -> lower=-3.14 upper=3.14 effort=5 velocity=0
- joint middle_left_HeelJoint: limit lower=-3.14 upper=3.14 effort=0 velocity=0 -> lower=-3.14 upper=3.14 effort=5 velocity=0
- joint middle_left_HipJoint: limit lower=-3.14 upper=3.14 effort=0 velocity=0 -> lower=-3.14 upper=3.14 effort=5 velocity=0
- joint middle_left_KneeJoint: limit lower=-3.14 upper=3.14 effort=0 velocity=0 -> lower=-3.14 upper=3.14 effort=5 velocity=0
- joint middle_right_HeelJoint: limit lower=-3.14 upper=3.14 effort=0 velocity=0 -> lower=-3.14 upper=3.14 effort=5 velocity=0
- joint middle_right_HipJoint: limit lower=-3.14 upper=3.14 effort=0 velocity=0 -> lower=-3.14 upper=3.14 effort=5 velocity=0
- joint middle_right_KneeJoint: limit lower=-3.14 upper=3.14 effort=0 velocity=0 -> lower=-3.14 upper=3.14 effort=5 velocity=0
- joint rear_left_HeelJoint: limit lower=-3.14 upper=3.14 effort=0 velocity=0 -> lower=-3.14 upper=3.14 effort=5 velocity=0
- joint rear_left_HipJoint: limit lower=-3.14 upper=3.14 effort=0 velocity=0 -> lower=-3.14 upper=3.14 effort=5 velocity=0
- joint rear_left_KneeJoint: limit lower=-3.14 upper=3.14 effort=0 velocity=0 -> lower=-3.14 upper=3.14 effort=5 velocity=0
- joint rear_right_HeelJoint: limit lower=-3.14 upper=3.14 effort=0 velocity=0 -> lower=-3.14 upper=3.14 effort=5 velocity=0
- joint rear_right_HipJoint: limit lower=-3.14 upper=3.14 effort=0 velocity=0 -> lower=-3.14 upper=3.14 effort=5 velocity=0
- joint rear_right_KneeJoint: limit lower=-3.14 upper=3.14 effort=0 velocity=0 -> lower=-3.14 upper=3.14 effort=5 velocity=0
